File: Merged Control Board/Maslow Mini Merged Board.kicad_sch (KiCad schematic)
At the start: 0 parts

Commit message: Merge
Other:
- note added: "+3V3 - one LM2596 (U116, 3 A) now feeds both sections. The driver board's 0.5 A MP2459 and its chain (U2, L3, D2, D6, C80, C81, R61-R63) are deleted;"
- note added: "Also removed as redundant: D101 + R115 (second power-on LED; LED2 + R17 kept), and D102/D103 changed SS14 -> SS36 to match D7."
- note added: "D7 is kept and ORs the driver USB port's VBUS into the shared buck input, so either USB port can still power the board."
- note added: "Each section still has its own ESP32-S3, its own USB-C programming port and its own boot button."
- note added: "Kept separate on purpose: BOOT_MC / BOOT_DRV, the two USB-C ports, and the two MCUs themselves."
- note added: "One PCB. Both ESP32-S3 MCUs are retained and meet only on the BoardCom pair below - everything else about the two"
- note added: "RST - one EN net. SW2 resets both MCUs; R28 (10k) + C134 (1 uF) are the single RC. R128 and C30 deleted."
- note added: "SHARED ACROSS BOTH SECTIONS"
- note added: "The 2x5 board-to-board header (H1 on both boards) is gone. Its four signal pins become the two BoardCom nets;"
- note added: "VIN (XT60 input, was H1 pins 6/8/10) - GND (was H1 pins 5/7/9)"
- note added: "its power pins (VIN x3, GND x3) become shared VIN and GND rails spanning both sections."
- note added: "original circuits is unchanged, apart from the redundancy that a single board makes pointless."
- note removed: "(+3V3_MC and +3V3_DRV are two different nets)."
- note removed: "Everything else stays separate - in particular each section keeps its own ESP32-S3, its own USB-C port and its own 3.3 V regulator"
- note removed: "One PCB, the two original circuits kept intact side by side."
- note removed: "Renamed to stay separate: 3V3 -> +3V3_MC / +3V3_DRV, BOOT -> BOOT_MC / BOOT_DRV."
- note removed: "Shared across both sections: VIN (XT60 input, was H1 pins 6/8/10) and GND (was H1 pins 5/7/9)."
- note removed: "The 2x5 board-to-board header (H1 on both boards) is gone. Its four signal pins become the two BoardCom nets below;"
- note removed: "its power pins (VIN x3, GND x3) become the shared VIN and GND rails, which now simply span both sections."
Changed lines of the file:
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@@
 		)
 	)
-	(text "One PCB, the two original circuits kept intact side by side."
+	(text "One PCB.  Both ESP32-S3 MCUs are retained and meet only on the BoardCom pair below - everything else about the two"
 		(at 25 38 0)
 		(effects
@@
 		)
 	)
-	(text "The 2x5 board-to-board header (H1 on both boards) is gone.  Its four signal pins become the two BoardCom nets below;"
-		(at 25 46 0)
-		(effects
-			(font
-				(size 2.0 2.0)
-			)
-			(justify left bottom)
-		)
-	)
-	(text "its power pins (VIN x3, GND x3) become the shared VIN and GND rails, which now simply span both sections."
-		(at 25 52 0)
-		(effects
-			(font
-				(size 2.0 2.0)
-			)
-			(justify left bottom)
-		)
-	)
-	(text "Everything else stays separate - in particular each section keeps its own ESP32-S3, its own USB-C port and its own 3.3 V regulator"
-		(at 25 58 0)
-		(effects
-			(font
-				(size 2.0 2.0)
-			)
-			(justify left bottom)
-		)
-	)
-	(text "(+3V3_MC and +3V3_DRV are two different nets)."
-		(at 25 64 0)
+	(text "original circuits is unchanged, apart from the redundancy that a single board makes pointless."
+		(at 25 44 0)
+		(effects
+			(font
+				(size 2.2 2.2)
+			)
+			(justify left bottom)
+		)
+	)
+	(text "The 2x5 board-to-board header (H1 on both boards) is gone.  Its four signal pins become the two BoardCom nets;"
+		(at 25 53 0)
+		(effects
+			(font
+				(size 2.0 2.0)
+			)
+			(justify left bottom)
+		)
+	)
+	(text "its power pins (VIN x3, GND x3) become shared VIN and GND rails spanning both sections."
+		(at 25 59 0)
+		(effects
+			(font
+				(size 2.0 2.0)
+			)
+			(justify left bottom)
+		)
+	)
+	(text "Each section still has its own ESP32-S3, its own USB-C programming port and its own boot button."
+		(at 25 65 0)
 		(effects
 			(font
@@
 		)
 	)
-	(text "Shared across both sections:  VIN (XT60 input, was H1 pins 6/8/10)  and  GND (was H1 pins 5/7/9)."
+	(text "SHARED ACROSS BOTH SECTIONS"
 		(at 25 165 0)
 		(effects
 			(font
-				(size 2.0 2.0)
-			)
-			(justify left bottom)
-		)
-	)
-	(text "Renamed to stay separate:  3V3 -> +3V3_MC / +3V3_DRV,  BOOT -> BOOT_MC / BOOT_DRV."
+				(size 2.4 2.4)
+				(bold yes)
+			)
+			(justify left bottom)
+		)
+	)
+	(text "VIN (XT60 input, was H1 pins 6/8/10)   -   GND (was H1 pins 5/7/9)"
 		(at 25 172 0)
 		(effects
@@
 		)
 	)
+	(text "+3V3   -   one LM2596 (U116, 3 A) now feeds both sections.  The driver board's 0.5 A MP2459 and its chain (U2, L3, D2, D6, C80, C81, R61-R63) are deleted;"
+		(at 25 178 0)
+		(effects
+			(font
+				(size 2.0 2.0)
+			)
+			(justify left bottom)
+		)
+	)
+	(text "            D7 is kept and ORs the driver USB port's VBUS into the shared buck input, so either USB port can still power the board."
+		(at 25 184 0)
+		(effects
+			(font
+				(size 2.0 2.0)
+			)
+			(justify left bottom)
+		)
+	)
+	(text "RST   -   one EN net.  SW2 resets both MCUs; R28 (10k) + C134 (1 uF) are the single RC.  R128 and C30 deleted."
+		(at 25 190 0)
+		(effects
+			(font
+				(size 2.0 2.0)
+			)
+			(justify left bottom)
+		)
+	)
+	(text "Also removed as redundant:  D101 + R115 (second power-on LED; LED2 + R17 kept), and D102/D103 changed SS14 -> SS36 to match D7."
+		(at 25 196 0)
+		(effects
+			(font
+				(size 2.0 2.0)
+			)
+			(justify left bottom)
+		)
+	)
+	(text "Kept separate on purpose:  BOOT_MC / BOOT_DRV, the two USB-C ports, and the two MCUs themselves."
+		(at 25 205 0)
+		(effects
+			(font
+				(size 2.0 2.0)
+			)
+			(justify left bottom)
+		)
+	)
 	(text "Motor-section reference designators are the originals + 100 (U2 -> U102, ...) so they do not collide with the driver section."
-		(at 25 179 0)
-		(effects
-			(font
+		(at 25 211 0)
+		(effects
+			(font
