File: Merged Control Board/driver_section.kicad_sch (KiCad schematic)
At the start: 88 parts, among them CN3 B3B-XH-2(LF)(SN), CN4 B3B-XH-2(LF)(SN), CN5 B3B-XH-2(LF)(SN), SW2 TSA002A3512A02, SW3 TSA002A3512A02, U12 2.4GHz, U14 MP6541A, U15 MP6541A, U2 MP2459GJ-Z

Commit message: Merge
Parts:
- removed C30: 100nF, ProPrj_Dri-easyedapro:C0402, symbol ProPrj_Dri-easyedapro:CL05B104KB54PNC
- removed C80: 10uF/50V, ProPrj_Dri-easyedapro:C0805, symbol ProPrj_Dri-easyedapro:GRM21BR61H106KE43L
- removed C81: 100nF/50V, ProPrj_Dri-easyedapro:C0603, symbol ProPrj_Dri-easyedapro:CL05B104KB54PNC
- removed D2, D6: SS36, Diode_SMD:D_SMA, symbol ProPrj_Dri-easyedapro:SS36
- removed L3: 47uH, Inductor_SMD:L_Bourns_SRN6045TA, symbol ProPrj_Dri-easyedapro:PRS3015-470MT
- removed R61: 124kΩ, ProPrj_Dri-easyedapro:R0402, symbol ProPrj_Dri-easyedapro:0402WGF1003TCE
- removed R62: 40.2kΩ, ProPrj_Dri-easyedapro:R0402, symbol ProPrj_Dri-easyedapro:0402WGF1002TCE
- removed R63: 100kΩ, ProPrj_Dri-easyedapro:R0402, symbol ProPrj_Dri-easyedapro:0402WGF1003TCE
- removed U2: MP2459GJ-Z, Package_TO_SOT_SMD:SOT-23-6, symbol ProPrj_Dri-easyedapro:MP2459
Connections:
- net +3V3_DRV renamed +3V3
Other:
- note added: "- 3V3 -> +3V3 and BOOT -> BOOT_DRV. +3V3, VIN, GND and RST are shared with the motor section; BOOT is not"
- note added: "- C30 deleted; R28 + SW2 + C134 (1 uF, motor section) are now the EN RC and reset button for BOTH MCUs"
- note added: "- D7 kept, and now ORs this port's VBUS into the shared buck input VIN_BUCK"
- note added: "- MP2459 buck chain (U2, L3, D2, D6, C80, C81, R61-R63) deleted - the motor section's 3 A LM2596 now feeds both sections"
- note added: "3.3 V DECOUPLING"
- note added: "Imported from "ProPrj_Driver Board to share_2026-08-01", except:"
- note added: "Regulator is now U116 (LM2596-3.3) on the motor section"
- note removed: "- 3V3 -> +3V3_DRV and BOOT -> BOOT_DRV, to stay distinct from the motor section"
- note removed: "- VIN and GND unchanged, and now merge with the motor section (they are what H1 pins 6/8/10 and 5/7/9 carried)"
- note removed: "-PMOS gate VBUS pull-up to prevent reverse current to buck output -This provides low voltage drop BUCK starts at 3.3V default -Also prioritizes VBUS over BUCK"
- note removed: "200ma LDO / Power OR-ing with PMOS"
- note removed: "3.3V Regulator"
- note removed: "Imported unchanged from "ProPrj_Driver Board to share_2026-08-01", except:"
