File: Merged Control Board/motor_control_section.kicad_sch (KiCad schematic)
At the start: 81 parts, among them CN101 B2B-PH-K-S(LF)(SN), CN103 B2B-PH-K-S(LF)(SN), CN104 B2B-PH-K-S(LF)(SN), CN105 B4B-PH-K-S(LF)(SN), CN109 B4B-PH-K-S(LF)(SN), CN110 B2B-PH-K-S(LF)(SN), CN111 B4B-PH-K-S(LF)(SN), CN112 B4B-PH-K-S(LF)(SN), SW101 DTSL-61N-V-T/R, U101 XT60PB-M.G.Y, U102 DRV8876PWPR, U103 DRV8876PWPR, U105 DRV8876PWPR, U106 DRV8876PWPR, U107 TCA9546A, U109 ZDSD01GLGEAG, U110 ESP32-S3-WROOM-1, U116 LM2596R-3.3

Commit message: Merge
Parts:
- removed D101: verde, MaslowMerged:LED0603-R-RD, symbol MaslowMerged:LED_A1K2
- removed R115: 120Ω, MaslowMerged:R0603, symbol MaslowMerged:R
- removed R128: 10K, MaslowMerged:R0603, symbol MaslowMerged:R
- D102, D103: value SS14 -> SS36; footprint MaslowMerged:SMA_L4.2-W2.6-LS5.3-RD -> Diode_SMD:D_SMA; symbol MaslowMerged:D_Schottky_K1A2 -> ProPrj_Dri-easyedapro:SS36
Connections:
- net +3V3_MC renamed +3V3
- net MCU_RST_MC renamed RST
- net SW_BUCK_MC renamed SW_BUCK
- net VIN_BUCK_MC renamed VIN_BUCK
Other:
- note added: "Derived from "Four Motor Control Board M5" - that board ships as a PCB with no schematic, so this sheet is reconstructed from its netlist. H1 removed; BoardCom is the hierarchical link to the driver section."
- note added: "VCC -> VIN and 3V3 -> +3V3: this LM2596 now feeds BOTH sections and the driver's 0.5 A MP2459 is deleted. R28/D1/R15 deleted as redundant. Reference designators are the originals + 100."
- note removed: "Derived from "Four Motor Control Board M5" - that board ships as a PCB with no schematic, so this sheet is reconstructed from its netlist. H1 (2x5 board-to-board header) removed; BoardCom is now the hierarchical link to the driver section. VCC renamed VIN and 3V3 renamed +3V3_MC. Reference designators are the originals + 100."
- moved on the sheet: C107, C108, C109, C110, C111, C112, C113, C114, C115, C116, C117, C118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
